Commit message: urdf方向修正

File: ros2_ws/src/t1_robot/t1_description/urdf/t1.urdf (robot description, URDF)
Before this commit: robot t1, 26 links, 25 joints
Joints:
- joint ARM-L-J1_Joint: axis 0 -1 0 -> 0 1 0
- joint ARM-L-J5_Joint: axis -1 0 0 -> 1 0 0
- joint ARM-L-J6_Joint: axis 0 0 -1 -> 0 0 1
- joint ARM-R-J2_Joint: axis -1 0 0 -> 1 0 0
- joint ARM-R-J4_Joint: axis 0 1 0 -> 0 -1 0
- joint ARM-R-J5_Joint: axis -1 0 0 -> 1 0 0
- joint ARM-R-J6_Joint: axis 0 0 -1 -> 0 0 1

Commit message: moveit控制器对接

File: ros2_ws/src/t1_robot/t1_description/urdf/t1.urdf (robot description, URDF)
Before this commit: robot t1, 26 links, 25 joints
Joints:
- joint ARM-L-J1_Joint: limit lower=-1.57 upper=2.09 effort=0 velocity=0 -> lower=-2.09 upper=1.57 effort=0 velocity=0
- joint ARM-R-J1_Joint: limit lower=-1.57 upper=2.09 effort=0 velocity=0 -> lower=-2.09 upper=1.57 effort=0 velocity=0
- joint ARM-R-J2_Joint: limit lower=-0.12 upper=2.61 effort=0 velocity=0 -> lower=-2.61 upper=0.12 effort=0 velocity=0
- joint ARM-R-J4_Joint: limit lower=-0.34 upper=3.14 effort=0 velocity=0 -> lower=-3.14 upper=0.34 effort=0 velocity=0

Commit message: urdf修改

File: ros2_ws/src/t1_robot/t1_description/urdf/t1.urdf (robot description, URDF)
Before this commit: robot t1, 26 links, 25 joints
Links:
- removed link ARM-R-J7_LINK
- added link ARM-R-J7_Link, mass 0.146890149456218; collision mesh filename=package://t1_description/meshes/ARM-R-J7_Link.STL; visual mesh filename=package://t1_description/meshes/ARM-R-J7_Link.STL
Joints:
- joint ARM-R-J7_Joint: child ARM-R-J7_LINK -> ARM-R-J7_Link

Commit message: urdf修改

File: ros2_ws/src/t1_robot/t1_description/urdf/t1.urdf (robot description, URDF)
Before this commit: robot t1, 26 links, 25 joints
Links:
- link ARM-L-J7_Link: geometry collision box size=0.15 0.24 0.24; collision mesh filename=package://t1_description/meshes/ARM-L-J7_Link.STL
- link ARM-R-J7_Link: geometry collision box size=0.15 0.24 0.24; collision mesh filename=package://t1_description/meshes/ARM-R-J7_Link.STL
Joints:
- joint SJ_Joint: origin xyz=0.13104 0 0.775 rpy=0 0 0 -> xyz=0.13104 0 0.725 rpy=0 0 0

Commit message: fix: expand arm joint limits to accommodate hardware tolerance

File: ros2_ws/src/t1_robot/t1_description/urdf/t1.urdf (robot description, URDF)
Before this commit: robot t1, 26 links, 25 joints
Joints:
- joint ARM-L-J1_Joint: limit lower=-2.09 upper=1.57 effort=0 velocity=0 -> lower=-2.18 upper=1.66 effort=0 velocity=0
- joint ARM-L-J2_Joint: limit lower=-0.12 upper=2.61 effort=0 velocity=0 -> lower=-0.21 upper=2.71 effort=0 velocity=0
- joint ARM-L-J4_Joint: limit lower=-0.34 upper=3.14 effort=0 velocity=0 -> lower=-0.44 upper=3.14 effort=0 velocity=0
- joint ARM-L-J7_Joint: limit lower=-1.48 upper=1.48 effort=0 velocity=0 -> lower=-1.57 upper=1.57 effort=0 velocity=0
- joint ARM-R-J1_Joint: limit lower=-2.09 upper=1.57 effort=0 velocity=0 -> lower=-2.18 upper=1.66 effort=0 velocity=0
- joint ARM-R-J2_Joint: limit lower=-2.61 upper=0.12 effort=0 velocity=0 -> lower=-2.71 upper=0.21 effort=0 velocity=0
- joint ARM-R-J4_Joint: limit lower=-3.14 upper=0.34 effort=0 velocity=0 -> lower=-3.14 upper=0.44 effort=0 velocity=0
- joint ARM-R-J7_Joint: limit lower=-1.48 upper=1.48 effort=0 velocity=0 -> lower=-1.57 upper=1.57 effort=0 velocity=0
