Commit message: urdf添加底盘碰撞体积

File: ros2_ws/src/t1_robot/t1_description/urdf/t1.urdf (robot description, URDF)
Before this commit: robot t1, 26 links, 25 joints
Links:
- link base_link: geometry collision box size=0.35 0.1 0.3; collision box size=0.5 0.1 0.3

Commit message: urdf限位更新

File: ros2_ws/src/t1_robot/t1_description/urdf/t1.urdf (robot description, URDF)
Before this commit: robot t1, 26 links, 25 joints
Joints:
- joint ARM-L-J1_Joint: limit lower=-2.18 upper=1.66 effort=0 velocity=0 -> lower=-2.0944 upper=1.5708 effort=0 velocity=0
- joint ARM-L-J2_Joint: limit lower=-0.21 upper=2.71 effort=0 velocity=0 -> lower=-0.1222 upper=2.7053 effort=0 velocity=0
- joint ARM-L-J3_Joint: limit lower=-3.05 upper=3.05 effort=0 velocity=0 -> lower=-3.1416 upper=3.1416 effort=0 velocity=0
- joint ARM-L-J4_Joint: limit lower=-0.44 upper=3.14 effort=0 velocity=0 -> lower=-0.3491 upper=3.1416 effort=0 velocity=0
- joint ARM-L-J5_Joint: limit lower=-3.05 upper=3.05 effort=0 velocity=0 -> lower=-3.1416 upper=3.1416 effort=0 velocity=0
- joint ARM-L-J6_Joint: limit lower=-0.52 upper=0.52 effort=0 velocity=0 -> lower=-0.5236 upper=0.5236 effort=0 velocity=0
- joint ARM-L-J7_Joint: limit lower=-1.57 upper=1.57 effort=0 velocity=0 -> lower=-1.4835 upper=1.4835 effort=0 velocity=0
- joint ARM-R-J1_Joint: limit lower=-2.18 upper=1.66 effort=0 velocity=0 -> lower=-1.5708 upper=2.0944 effort=0 velocity=0
- joint ARM-R-J2_Joint: limit lower=-2.71 upper=0.21 effort=0 velocity=0 -> lower=-2.7053 upper=0.1222 effort=0 velocity=0
- joint ARM-R-J3_Joint: limit lower=-3.05 upper=3.05 effort=0 velocity=0 -> lower=-3.0543 upper=3.0543 effort=0 velocity=0
- joint ARM-R-J4_Joint: limit lower=-3.14 upper=0.44 effort=0 velocity=0 -> lower=-3.1416 upper=0.3491 effort=0 velocity=0
- joint ARM-R-J5_Joint: limit lower=-3.05 upper=3.05 effort=0 velocity=0 -> lower=-3.0543 upper=3.0543 effort=0 velocity=0
- joint ARM-R-J6_Joint: limit lower=-0.52 upper=0.52 effort=0 velocity=0 -> lower=-0.5236 upper=0.5236 effort=0 velocity=0
- joint ARM-R-J7_Joint: limit lower=-1.57 upper=1.57 effort=0 velocity=0 -> lower=-1.4835 upper=1.4835 effort=0 velocity=0

Commit message: urdf修改,增大碰撞体积

File: ros2_ws/src/t1_robot/t1_description/urdf/t1.urdf (robot description, URDF)
Before this commit: robot t1, 26 links, 25 joints
Links:
- link ARM-L-J7_Link: geometry collision box size=0.3 0.24 0.24; collision mesh filename=package://t1_description/meshes/ARM-L-J7_Link.STL
- link ARM-R-J7_Link: geometry collision box size=0.3 0.24 0.24; collision mesh filename=package://t1_description/meshes/ARM-R-J7_Link.STL
- link base_link: geometry collision box size=0.75 0.1 0.3; collision box size=0.75 0.1 0.3
